File: LightArm/3 channel RGB MOSFET board/KiCad/3ChanMosfetBoard.sch (KiCad schematic (older format))
At the start: 20 parts, among them IC1 MOC3010M, IC2 MOC3010M, IC3 MOC3010M, K1 CONN_3, P1 PWM, P2 CONN_2, P3 CONN_2, P4 CONN_2, Q1 C_MOS, Q2 C_MOS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

Commit message: update light and motor boards
Parts:
- removed IC1, IC2, IC3: MOC3010M, DIP6, symbol MOC3010M
- added IC1, IC2, IC3: CPMOC, DIP4, symbol CPMOC
- Q1, Q2, Q3: symbol C_MOS -> c_mos
Connections:
- wire segments 77 -> 69
Other:
- moved on the sheet: R1, R2, R3
Changed lines of the file:
@@
 EESchema Schematic File Version 2
-LIBS:power
-LIBS:device
-LIBS:transistors
-LIBS:conn
-LIBS:linear
-LIBS:regul
-LIBS:74xx
-LIBS:cmos4000
-LIBS:adc-dac
-LIBS:memory
-LIBS:xilinx
-LIBS:special
-LIBS:microcontrollers
-LIBS:dsp
-LIBS:microchip
-LIBS:analog_switches
-LIBS:motorola
-LIBS:texas
-LIBS:intel
-LIBS:audio
-LIBS:interface
-LIBS:digital-audio
-LIBS:philips
-LIBS:display
-LIBS:cypress
-LIBS:siliconi
-LIBS:opto
-LIBS:atmel
-LIBS:contrib
-LIBS:valves
+LIBS:3ChanMosfetBoard-rescue
 LIBS:ECA
 LIBS:Chris
 LIBS:3ChanMosfetBoard-cache
-EELAYER 27 0
+EELAYER 25 0
 EELAYER END
 $Descr A4 11693 8268
@@
 Sheet 1 1
 Title ""
-Date "9 aug 2017"
+Date "18 aug 2017"
 Rev ""
 Comp ""
@@
 L R R1
 U 1 1 596E543C
-P 3200 2450
-F 0 "R1" V 3280 2450 40  0000 C CNN
-F 1 "R500" V 3207 2451 40  0000 C CNN
-F 2 "~" V 3130 2450 30  0000 C CNN
-F 3 "~" H 3200 2450 30  0000 C CNN
-	1    3200 2450
-	-1   0    0    1
+P 3150 1900
+F 0 "R1" V 3230 1900 40  0000 C CNN
+F 1 "R500" V 3157 1901 40  0000 C CNN
+F 2 "~" V 3080 1900 30  0000 C CNN
+F 3 "~" H 3150 1900 30  0000 C CNN
+	1    3150 1900
+	0    1    1    0
 $EndComp
 $Comp
 L R R2
 U 1 1 596E544B
-P 3050 2350
-F 0 "R2" V 3130 2350 40  0000 C CNN
-F 1 "R500" V 3057 2351 40  0000 C CNN
-F 2 "~" V 2980 2350 30  0000 C CNN
-F 3 "~" H 3050 2350 30  0000 C CNN
-	1    3050 2350
-	-1   0    0    1
+P 3150 2350
+F 0 "R2" V 3230 2350 40  0000 C CNN
+F 1 "R500" V 3157 2351 40  0000 C CNN
+F 2 "~" V 3080 2350 30  0000 C CNN
+F 3 "~" H 3150 2350 30  0000 C CNN
+	1    3150 2350
+	0    1    1    0
 $EndComp
 $Comp
 L R R3
 U 1 1 596E545A
-P 3300 2900
-F 0 "R3" V 3380 2900 40  0000 C CNN
-F 1 "R500" V 3307 2901 40  0000 C CNN
-F 2 "~" V 3230 2900 30  0000 C CNN
-F 3 "~" H 3300 2900 30  0000 C CNN
-	1    3300 2900
-	-1   0    0    1
+P 3150 2800
+F 0 "R3" V 3230 2800 40  0000 C CNN
+F 1 "R500" V 3157 2801 40  0000 C CNN
+F 2 "~" V 3080 2800 30  0000 C CNN
+F 3 "~" H 3150 2800 30  0000 C CNN
+	1    3150 2800
+	0    1    1    0
 $EndComp
 Wire Wire Line
 	2650 2450 2650 3000
 Wire Wire Line
-	2900 2350 3450 2350
-Wire Wire Line
 	2650 2150 2900 2150
 Wire Wire Line
@@
 	2650 2350 2800 2350
 Wire Wire Line
-	2800 2350 2800 2500
-Wire Wire Line
-	2800 2500 2900 2500
-Wire Wire Line
-	2900 2500 2900 2800
-Wire Wire Line
-	3050 2100 3450 2100
+	2800 2350 2800 2800
 $Comp
 L R R4
@@
 Connection ~ 4900 2800
 Connection ~ 4900 2350
-Connection ~ 4900 3250
 Wire Wire Line
 	4900 3250 5350 3250
@@
 	4950 1650 6800 1650
 Connection ~ 6250 1650
-Wire Wire Line
-	2900 2800 3450 2800
-Wire Wire Line
-	2900 1900 3450 1900
 $Comp
 L ECA C1
@@
 	5050 3150 5650 3150
 $Comp
-L MOC3010M IC1
-U 1 1 59724009
-P 3800 2000
-F 0 "IC1" H 3590 2190 40  0000 C CNN
-F 1 "MOC3010M" H 3900 1810 40  0000 C CNN
-F 2 "DIP6" H 3600 1820 30  0000 C CIN
-F 3 "~" H 3800 2000 60  0000 C CNN
-	1    3800 2000
-	1    0    0    -1
-$EndComp
-$Comp
-L MOC3010M IC2
-U 1 1 59724018
-P 3800 2450
-F 0 "IC2" H 3590 2640 40  0000 C CNN
-F 1 "MOC3010M" H 3900 2260 40  0000 C CNN
-F 2 "DIP6" H 3600 2270 30  0000 C CIN
-F 3 "~" H 3800 2450 60  0000 C CNN
-	1    3800 2450
-	1    0    0    -1
-$EndComp
-$Comp
-L MOC3010M IC3
-U 1 1 59724027
-P 3800 2900
-F 0 "IC3" H 3590 3090 40  0000 C CNN
-F 1 "MOC3010M" H 3900 2710 40  0000 C CNN
-F 2 "DIP6" H 3600 2720 30  0000 C CIN
-F 3 "~" H 3800 2900 60  0000 C CNN
-	1    3800 2900
-	1    0    0    -1
-$EndComp
-$Comp
-L C_MOS Q1
+L c_mos Q1
 U 1 1 597241D0
 P 5550 1950
@@
 $EndComp
 $Comp
-L C_MOS Q2
+L c_mos Q2
 U 1 1 597241DF
 P 5550 2450
@@
 $EndComp
 $Comp
-L C_MOS Q3
+L c_mos Q3
 U 1 1 597241EE
 P 5550 2950
@@
 $EndComp
 Wire Wire Line
-	3450 2550 3350 2550
-Wire Wire Line
-	3350 2550 3350 2200
-Wire Wire Line
-	3350 2200 3200 2200
-Wire Wire Line
-	3450 3000 3400 3000
-Wire Wire Line
-	3400 3000 3400 2650
-Wire Wire Line
-	3400 2650 3300 2650
-Wire Wire Line
-	2650 3000 3200 3000
-Wire Wire Line
-	3200 2700 3200 3150
-Wire Wire Line
-	3200 3150 3300 3150
-Connection ~ 3200 3000
-Wire Wire Line
-	3050 2600 3050 3000
-Connection ~ 3050 3000
+	2650 3000 3450 3000
+Wire Wire Line
+	3350 2550 3450 2550
+Wire Wire Line
+	3400 2350 3450 2350
+Wire Wire Line
+	3350 2100 3450 2100
+Wire Wire Line
+	3400 1900 3450 1900
+Wire Wire Line
+	2800 2800 2900 2800
+Wire Wire Line
+	3400 2800 3450 2800
+Wire Wire Line
+	3350 2100 3350 3000
+Connection ~ 3350 3000
+Connection ~ 3350 2550
+$Comp
+L CPMOC IC1
+U 1 1 59976F4D
+P 3800 2000
+F 0 "IC1" H 3590 2190 40  0000 C CNN
+F 1 "CPMOC" H 3900 1810 40  0000 C CNN
+F 2 "DIP4" H 3600 1820 30  0000 C CIN
+F 3 "~" H 3800 2000 60  0000 C CNN
+	1    3800 2000
+	1    0    0    -1
+$EndComp
+$Comp
+L CPMOC IC2
+U 1 1 59976F5C
+P 3800 2450
+F 0 "IC2" H 3590 2640 40  0000 C CNN
+F 1 "CPMOC" H 3900 2260 40  0000 C CNN
+F 2 "DIP4" H 3600 2270 30  0000 C CIN
+F 3 "~" H 3800 2450 60  0000 C CNN
+	1    3800 2450
+	1    0    0    -1
+$EndComp
+$Comp
+L CPMOC IC3
+U 1 1 59976F6B
+P 3800 2900
+F 0 "IC3" H 3590 3090 40  0000 C CNN
+F 1 "CPMOC" H 3900 2710 40  0000 C CNN
+F 2 "DIP4" H 3600 2720 30  0000 C CIN
+F 3 "~" H 3800 2900 60  0000 C CNN
+	1    3800 2900
+	1    0    0    -1
+$EndComp
 $EndSCHEMATC

Commit message: updating various changes in codebase , adding in new esp32 directory for code running on the esp32
Parts:
- R1, R2, R3, R4, R5, R6: symbol R -> R-RESCUE-3ChanMosfetBoard
Changed lines of the file:
@@
 EESchema Schematic File Version 2
 LIBS:3ChanMosfetBoard-rescue
+LIBS:power
+LIBS:device
+LIBS:transistors
+LIBS:conn
+LIBS:linear
+LIBS:regul
+LIBS:74xx
+LIBS:cmos4000
+LIBS:adc-dac
+LIBS:memory
+LIBS:xilinx
+LIBS:microcontrollers
+LIBS:dsp
+LIBS:microchip
+LIBS:analog_switches
+LIBS:motorola
+LIBS:texas
+LIBS:intel
+LIBS:audio
+LIBS:interface
+LIBS:digital-audio
+LIBS:philips
+LIBS:display
+LIBS:cypress
+LIBS:siliconi
+LIBS:opto
+LIBS:atmel
+LIBS:contrib
+LIBS:valves
 LIBS:ECA
 LIBS:Chris
@@
 $EndComp
 $Comp
-L R R1
+L R-RESCUE-3ChanMosfetBoard R1
 U 1 1 596E543C
 P 3150 1900
@@
 $EndComp
 $Comp
-L R R2
+L R-RESCUE-3ChanMosfetBoard R2
 U 1 1 596E544B
 P 3150 2350
@@
 $EndComp
 $Comp
-L R R3
+L R-RESCUE-3ChanMosfetBoard R3
 U 1 1 596E545A
 P 3150 2800
@@
 	2800 2350 2800 2800
 $Comp
-L R R4
+L R-RESCUE-3ChanMosfetBoard R4
 U 1 1 596E5521
 P 4600 1900
@@
 $EndComp
 $Comp
-L R R5
+L R-RESCUE-3ChanMosfetBoard R5
 U 1 1 596E5530
 P 4600 2350
@@
 $EndComp
 $Comp
-L R R6
+L R-RESCUE-3ChanMosfetBoard R6
 U 1 1 596E553F
 P 4600 2800
